File: stepper_board.sch (EAGLE design)
At the start: 79 parts

Commit message: Slight change to a capacitor value
Parts:
- C31: value 100n -> 0.1u
Changed lines of the file:
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@@
 <part name="TP4" library="testpad" deviceset="PTR1" device="B1,27"/>
 <part name="RST" library="switch-omron" deviceset="10-XX" device=""/>
-<part name="C31" library="rcl" deviceset="C-US" device="C0805" value="100n"/>
+<part name="C31" library="rcl" deviceset="C-US" device="C0805" value="0.1u"/>
 <part name="GND19" library="supply1" deviceset="GND" device=""/>
 <part name="+3V10" library="supply1" deviceset="+3V3" device=""/>
